File: Final/oscillator/oscillator/oscillator.sch (KiCad schematic (older format))
At the start: 54 parts, among them J1 V15V_IN, J2 V15V_IN, J3 Select, J4 SQ Out, J5 TRI Out, J6 SQ Out, J7 TRI Out, SW1 SS-10-16NPE, SW2 SW_SPDT, U1 LM6172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

Commit message: 
Connections:
- net at R3.1, R5.2, SW1.C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: now also R1.1, U1.6 (-)
Other:
- note added: "Amplify Triangle Wave"
- note added: "Power Connections"
- note added: "Signal Generator - Oscillator Board"
- note removed: "Amplify Tri Wave"
- note removed: "Power Connection"
- moved on the sheet: C10, C11, C12, C13, C14, C15, C16, C17, C3, C4, C6, C7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
